File: cad-source-files/robo_car/robo_car.kicad_sch (KiCad schematic)
At the start: 86 parts, among them J1 Conn_01x06_MountingPin, J16 Conn_01x02_MountingPin, J2 ftdi_conn, J3 Conn_01x06_MountingPin, J4 Barrel_Jack, J5 Conn_01x04, J6 Conn_01x06_MountingPin, J7 Conn_01x02_MountingPin, J8 Conn_01x02_MountingPin, SW1 SW_Push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

Commit message: Revert "3rd try lets go"
This reverts commit 3f093a060dbc0dc4159fd1f3f57facfb81c75c62.
Connections:
- net IO13 renamed INPUT_D
- net IO16 renamed INPUT_A
- net IO17 renamed INPUT_B
- net IO4 renamed INPUT_C
Changed lines of the file:
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@@
     (effects (font (size 1.27 1.27)) (justify right bottom))
   )
-  (label "IO4" (at 41.91 129.54 0)
+  (label "INPUT_C" (at 41.91 129.54 0)
     (effects (font (size 1.27 1.27)) (justify left bottom))
   )
@@
     (effects (font (size 1.27 1.27)) (justify right bottom))
   )
-  (label "IO4" (at 311.15 152.4 180)
+  (label "INPUT_C" (at 311.15 152.4 180)
     (effects (font (size 1.27 1.27)) (justify right bottom))
   )
@@
     (effects (font (size 1.27 1.27)) (justify left bottom))
   )
-  (label "IO16" (at 41.91 127 0)
+  (label "INPUT_A" (at 41.91 127 0)
     (effects (font (size 1.27 1.27)) (justify left bottom))
   )
@@
     (effects (font (size 1.27 1.27)) (justify left bottom))
   )
-  (label "IO17" (at 316.23 170.18 180)
+  (label "INPUT_B" (at 316.23 170.18 180)
     (effects (font (size 1.27 1.27)) (justify right bottom))
   )
@@
     (effects (font (size 1.27 1.27)) (justify right bottom))
   )
-  (label "IO13" (at 314.96 160.02 180)
+  (label "INPUT_D" (at 314.96 160.02 180)
     (effects (font (size 1.27 1.27)) (justify right bottom))
   )
@@
     (effects (font (size 1.27 1.27)) (justify right bottom))
   )
-  (label "IO17" (at 41.91 124.46 0)
+  (label "INPUT_B" (at 41.91 124.46 0)
     (effects (font (size 1.27 1.27)) (justify left bottom))
   )
-  (label "IO16" (at 311.15 167.64 180)
+  (label "INPUT_A" (at 311.15 167.64 180)
     (effects (font (size 1.27 1.27)) (justify right bottom))
   )
@@
     (effects (font (size 1.27 1.27)) (justify left bottom))
   )
-  (label "IO13" (at 41.91 121.92 0)
+  (label "INPUT_D" (at 41.91 121.92 0)
     (effects (font (size 1.27 1.27)) (justify left bottom))
   )
