File: cad-source-files/robo_car/robo_car.kicad_sch (KiCad schematic)
At the start: 89 parts, among them J1 Conn_01x06_MountingPin, J16 Conn_01x02_MountingPin, J2 ftdi_conn, J3 Conn_01x06_MountingPin, J4 Barrel_Jack, J5 Conn_01x04, J6 Conn_01x06_MountingPin, J7 Conn_01x02_MountingPin, J8 Conn_01x02_MountingPin, J9 Conn_01x02_MountingPin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

Commit message: 12-2 boards ordered
Parts:
- added D2: SX35_SCHOTTKY, Diode_SMD:D_SMA, symbol Device:D_Schottky
Connections:
- net GND: now also D2.2 (A)
- net VBUS: now also D2.1 (K)
Other:
- moved on the sheet: J4, J9, SW3
Changed lines of the file:
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@@
   (junction (at 251.46 80.01) (diameter 1.016) (color 0 0 0 0)
   )
+  (junction (at 259.08 35.56) (diameter 0) (color 0 0 0 0)
+  )
   (junction (at 299.72 134.62) (diameter 1.016) (color 0 0 0 0)
   )
@@
     (stroke (width 0) (type solid) (color 0 0 0 0))
   )
-  (wire (pts (xy 238.76 49.53) (xy 243.84 49.53))
+  (wire (pts (xy 238.76 46.99) (xy 243.84 46.99))
     (stroke (width 0) (type default) (color 0 0 0 0))
   )
@@
     (stroke (width 0) (type solid) (color 0 0 0 0))
   )
+  (wire (pts (xy 259.08 33.02) (xy 259.08 35.56))
+    (stroke (width 0) (type default) (color 0 0 0 0))
+  )
   (wire (pts (xy 394.97 177.8) (xy 400.05 177.8))
     (stroke (width 0) (type solid) (color 0 0 0 0))
@@
     (stroke (width 0) (type default) (color 0 0 0 0))
   )
-  (wire (pts (xy 243.84 49.53) (xy 243.84 40.64))
+  (wire (pts (xy 243.84 38.1) (xy 243.84 46.99))
     (stroke (width 0) (type default) (color 0 0 0 0))
   )
@@
     (stroke (width 0) (type solid) (color 0 0 0 0))
   )
-  (wire (pts (xy 238.76 35.56) (xy 243.84 35.56))
+  (wire (pts (xy 238.76 33.02) (xy 243.84 33.02))
     (stroke (width 0) (type default) (color 0 0 0 0))
   )
@@
     (stroke (width 0) (type default) (color 0 0 0 0))
   )
-  (wire (pts (xy 254 38.1) (xy 256.54 38.1))
+  (wire (pts (xy 254 35.56) (xy 259.08 35.56))
     (stroke (width 0) (type default) (color 0 0 0 0))
   )
@@
     (pin "1")
   )
-  (symbol (lib_id "power:VBUS") (at 256.54 38.1 0) (unit 1)
+  (symbol (lib_id "power:VBUS") (at 259.08 33.02 0) (unit 1)
     (in_bom yes) (on_board yes)
-    (property "Reference" "#PWR029" (id 0) (at 256.54 41.91 0)
+    (property "Reference" "#PWR029" (id 0) (at 259.08 36.83 0)
       (effects (font (size 1.27 1.27)) hide)
     )
-    (property "Value" "VBUS" (id 1) (at 256.54 33.02 90))
-    (property "Footprint" "" (id 2) (at 256.54 38.1 0)
+    (property "Value" "VBUS" (id 1) (at 259.08 27.94 90))
+    (property "Footprint" "" (id 2) (at 259.08 33.02 0)
       (effects (font (size 1.27 1.27)) hide)
     )
-    (property "Datasheet" "" (id 3) (at 256.54 38.1 0)
+    (property "Datasheet" "" (id 3) (at 259.08 33.02 0)
       (effects (font (size 1.27 1.27)) hide)
     )
@@
     (pin "1")
   )
-  (symbol (lib_id "power:GND") (at 238.76 38.1 0) (mirror y) (unit 1)
+  (symbol (lib_id "power:GND") (at 238.76 35.56 0) (mirror y) (unit 1)
     (in_bom yes) (on_board yes)
-    (property "Reference" "#PWR038" (id 0) (at 238.76 44.45 0)
+    (property "Reference" "#PWR038" (id 0) (at 238.76 41.91 0)
       (effects (font (size 1.27 1.27)) hide)
     )
-    (property "Value" "GND" (id 1) (at 238.633 42.4942 0))
-    (property "Footprint" "" (id 2) (at 238.76 38.1 0)
+    (property "Value" "GND" (id 1) (at 238.633 39.9542 0))
+    (property "Footprint" "" (id 2) (at 238.76 35.56 0)
       (effects (font (size 1.27 1.27)) hide)
     )
-    (property "Datasheet" "" (id 3) (at 238.76 38.1 0)
+    (property "Datasheet" "" (id 3) (at 238.76 35.56 0)
       (effects (font (size 1.27 1.27)) hide)
     )
@@
     )
   )
+  (symbol (lib_id "power:GND") (at 259.08 43.18 0) (unit 1)
+    (in_bom yes) (on_board yes)
+    (property "Reference" "#PWR040" (id 0) (at 259.08 49.53 0)
+      (effects (font (size 1.27 1.27)) hide)
+    )
+    (property "Value" "GND" (id 1) (at 259.207 47.5742 0))
+    (property "Footprint" "" (id 2) (at 259.08 43.18 0)
+      (effects (font (size 1.27 1.27)) hide)
+    )
+    (property "Datasheet" "" (id 3) (at 259.08 43.18 0)
+      (effects (font (size 1.27 1.27)) hide)
+    )
+    (pin "1")
+  )
   (symbol (lib_id "power:GND") (at 74.295 22.86 0) (mirror y) (unit 1)
     (in_bom yes) (on_board yes)
@@
     )
   )
-  (symbol (lib_id "power:GND") (at 238.76 54.61 0) (unit 1)
+  (symbol (lib_id "power:GND") (at 238.76 52.07 0) (unit 1)
     (in_bom yes) (on_board yes)
-    (property "Reference" "#PWR030" (id 0) (at 238.76 60.96 0)
+    (property "Reference" "#PWR030" (id 0) (at 238.76 58.42 0)
       (effects (font (size 1.27 1.27)) hide)
     )
-    (property "Value" "GND" (id 1) (at 238.887 59.0042 0))
-    (property "Footprint" "" (id 2) (at 238.76 54.61 0)
+    (property "Value" "GND" (id 1) (at 238.887 56.4642 0))
+    (property "Footprint" "" (id 2) (at 238.76 52.07 0)
       (effects (font (size 1.27 1.27)) hide)
     )
-    (property "Datasheet" "" (id 3) (at 238.76 54.61 0)
+    (property "Datasheet" "" (id 3) (at 238.76 52.07 0)
       (effects (font (size 1.27 1.27)) hide)
     )
@@
     )
   )
-  (symbol (lib_id "Connector_Generic_MountingPin:Conn_01x02_MountingPin") (at 233.68 35.56 0) (mirror y) (unit 1)
+  (symbol (lib_id "Connector_Generic_MountingPin:Conn_01x02_MountingPin") (at 233.68 33.02 0) (mirror y) (unit 1)
     (in_bom yes) (on_board yes)
-    (property "Reference" "J9" (id 0) (at 234.8229 32.8735 0)
+    (property "Reference" "J9" (id 0) (at 234.8229 30.3335 0)
       (effects (font (size 1.27 1.27)) (justify left))
     )
-    (property "Value" "Conn_01x02_MountingPin" (id 1) (at 231.0129 45.8086 90)
+    (property "Value" "Conn_01x02_MountingPin" (id 1) (at 231.0129 43.2686 90)
       (effects (font (size 0.75 0.75)) (justify left))
     )
-    (property "Footprint" "Connector_JST:JST_XH_B2B-XH-AM_1x02_P2.50mm_Vertical" (id 2) (at 233.68 35.56 0)
+    (property "Footprint" "Connector_JST:JST_XH_B2B-XH-AM_1x02_P2.50mm_Vertical" (id 2) (at 233.68 33.02 0)
       (effects (font (size 1.27 1.27)) hide)
     )
-    (property "Datasheet" "~" (id 3) (at 233.68 35.56 0)
+    (property "Datasheet" "~" (id 3) (at 233.68 33.02 0)
       (effects (font (size 1.27 1.27)) hide)
     )
@@
     (pin "2")
   )
-  (symbol (lib_id "Connector:Barrel_Jack") (at 231.14 52.07 0) (unit 1)
+  (symbol (lib_id "Connector:Barrel_Jack") (at 231.14 49.53 0) (unit 1)
     (in_bom yes) (on_board yes) (fields_autoplaced)
-    (property "Reference" "J4" (id 0) (at 231.14 43.18 0))
-    (property "Value" "Barrel_Jack" (id 1) (at 231.14 45.72 0))
-    (property "Footprint" "Connector_BarrelJack:BarrelJack_Horizontal" (id 2) (at 232.41 53.086 0)
+    (property "Reference" "J4" (id 0) (at 231.14 40.64 0))
+    (property "Value" "Barrel_Jack" (id 1) (at 231.14 43.18 0))
+    (property "Footprint" "Connector_BarrelJack:BarrelJack_Horizontal" (id 2) (at 232.41 50.546 0)
       (effects (font (size 1.27 1.27)) hide)
     )
-    (property "Datasheet" "~" (id 3) (at 232.41 53.086 0)
+    (property "Datasheet" "~" (id 3) (at 232.41 50.546 0)
       (effects (font (size 1.27 1.27)) hide)
     )
@@
     (pin "2")
   )
-  (symbol (lib_id "Switch:SW_SPDT") (at 248.92 38.1 0) (mirror y) (unit 1)
+  (symbol (lib_id "Switch:SW_SPDT") (at 248.92 35.56 0) (mirror y) (unit 1)
     (in_bom yes) (on_board yes) (fields_autoplaced)
-    (property "Reference" "SW3" (id 0) (at 248.92 30.48 0))
-    (property "Value" "SW_SPDT" (id 1) (at 248.92 33.02 0))
-    (property "Footprint" "Button_Switch_THT:SW_SLIDE_SS-12D10L9" (id 2) (at 248.92 38.1 0)
+    (property "Reference" "SW3" (id 0) (at 248.92 27.94 0))
+    (property "Value" "SW_SPDT" (id 1) (at 248.92 30.48 0))
+    (property "Footprint" "Button_Switch_THT:SW_SLIDE_SS-12D10L9" (id 2) (at 248.92 35.56 0)
       (effects (font (size 1.27 1.27)) hide)
     )
-    (property "Datasheet" "~" (id 3) (at 248.92 38.1 0)
+    (property "Datasheet" "~" (id 3) (at 248.92 35.56 0)
       (effects (font (size 1.27 1.27)) hide)
     )
@@
     )
   )
+  (symbol (lib_id "Device:D_Schottky") (at 259.08 39.37 270) (unit 1)
+    (in_bom yes) (on_board yes)
+    (property "Reference" "D2" (id 0) (at 261.0866 38.2016 90)
+      (effects (font (size 1.27 1.27)) (justify left))
+    )
+    (property "Value" "SX35_SCHOTTKY" (id 1) (at 262.89 40.64 90)
+      (effects (font (size 1.27 1.27)) (justify left))
+    )
+    (property "Footprint" "Diode_SMD:D_SMA" (id 2) (at 259.08 39.37 0)
+      (effects (font (size 1.27 1.27)) hide)
+    )
+    (property "Datasheet" "~" (id 3) (at 259.08 39.37 0)
+      (effects (font (size 1.27 1.27)) hide)
+    )
+    (pin "1")
+    (pin "2")
+  )
   (symbol (lib_id "LED:SK6812MINI") (at 111.76 229.87 0) (unit 1)
     (in_bom yes) (on_board yes)
@@
       (reference "#PWR039") (unit 1) (value "GND") (footprint "")
     )
+    (path "/71ac0761-e35f-4982-a617-c67ffde7418c"
+      (reference "#PWR040") (unit 1) (value "GND") (footprint "")
+    )
     (path "/a8235ac4-b0cf-46b7-9a6f-6bbd038c49c1"
       (reference "#PWR043") (unit 1) (value "VBUS") (footprint "")
@@
       (reference "D1") (unit 1) (value "SX35_SCHOTTKY") (footprint "Diode_SMD:D_SMA")
     )
+    (path "/f2fca0b6-1a6f-4d3f-b354-b2bb5cdb11be"
+      (reference "D2") (unit 1) (value "SX35_SCHOTTKY") (footprint "Diode_SMD:D_SMA")
+    )
     (path "/00000000-0000-0000-0000-00005f56b202"
