File: cad-source-files/accessory-boards/i2c_board/i2c_board.kicad_sch (KiCad schematic)
At the start: 11 parts, among them J9 Conn_01x06_MountingPin

Commit message: qwiic quick board
Parts:
- removed SW?: SW_Push, EvezorLIB:SWITCH_2x3_SMD_TACTILE_GREEN, symbol Switch:SW_Push
- added D1: led_g, LED_SMD:LED_0603_1608Metric, symbol Device:LED
- added R4: 10k, Resistor_SMD:R_0603_1608Metric, symbol Device:R_Small
- J1: renamed from J?; footprint (none) -> Connector_JST:JST_SH_SM04B-SRSS-TB_1x04-1MP_P1.00mm_Horizontal
- JP1, JP2: renamed from JP?; footprint (none) -> Jumper:SolderJumper-2_P1.3mm_Bridged_RoundedPad1.0x1.5mm
- R2, R3: renamed from R?; value 10k -> 4.7k
- SW1: renamed from SW?; footprint EvezorLIB:SWITCH_2x3_SMD_TACTILE_GREEN -> Button_Switch_SMD:SWITCH_2x3_SMD_TACTILE_GREEN
- gave numbers to parts that had none: 1
Connections:
- net FUNCTION_BUTTON is gone; now on net B: R1.1, SW1.1
- net SCL is gone; now on net C: J1.4 (Pin_4), JP1.1 (A)
- net SDA is gone; now on net D: J1.3 (Pin_3), JP2.1 (A)
- net A: now also J9.4 (Pin_4), R4.1; no longer J9.1 (Pin_1)
- net B: now also J9.3 (Pin_3); no longer J9.2 (Pin_2)
- net C: now also J9.2 (Pin_2); no longer J9.3 (Pin_3)
- net D: now also J9.1 (Pin_1); no longer J9.4 (Pin_4)
- net GND: now also D1.1 (K)
- new net: D1.2 (A), R4.2
Other:
- moved on the sheet: J9
