File: cad-source-files/accessory-boards/mo-stache/mo-stache.kicad_pcb (KiCad board)
At the start: 2 copper layers, 84.1 x 109.6 mm, 11 parts, among them J1 Conn_01x02

Commit message: mo can see us now 👀
Parts:
- added G***: LOGO, Symbol:Mustache20mm, B.Cu at (117.9, 131.0)
- moved H1 139.5 mm to (82.5, 155.0)
- moved H4 134.3 mm to (65.7, 93.0)
- moved H7 112.5 mm to (93.2, 93.0)
- moved H5 87.2 mm to (106.8, 93.0)
- moved H2 77.5 mm to (100.0, 155.0)
- turned BT1 to -90 degrees
- turned BT2 to 90 degrees
- turned BT3 to -90 degrees
Routing:
- net Net-(BT2-Pad2): track 0.00 -> 26.6 mm
- net Net-(BT1-Pad2): track 0.00 -> 19.0 mm
- net +BATT: track 0.00 -> 12.6 mm
- added copper zone on B.Cu, net GND
- added copper zone on F.Cu, net GND
Other:
- board text added: "+"
- board text added: "-"
- board text added: "Mo"
- board text added: "Olivia & Andrew 2022"
- board text added: "The Most Magnificent Mustached Machine"

Commit message: 12-2 boards ordered
Other:
- board text added: "made by:"
- board text added: "power output"
Changed lines of the file:
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@@
       (outputformat 1)
       (mirror false)
-      (drillshape 1)
+      (drillshape 0)
       (scaleselection 1)
-      (outputdirectory "")
+      (outputdirectory "../../../../../../Desktop/mo-stache/")
     )
   )
@@
     (fp_line (start 0 -1.35) (end 0.625 -2.35) (layer "F.Fab") (width 0.1))
     (pad "" np_thru_hole circle locked (at -1.6 2 270) (size 1.2 1.2) (drill 1.2) (layers *.Cu *.Mask))
-    (pad "1" thru_hole roundrect locked (at 0 0 270) (size 1.7 2) (drill 1) (layers *.Cu *.Mask) (roundrect_rratio 0.147059)
+    (pad "1" thru_hole roundrect locked (at 0 0 270) (size 1.7 2) (drill 1) (layers *.Cu *.Mask) (roundrect_rratio 0.1470588235)
       (net 1 "+BATT") (pinfunction "Pin_1") (pintype "passive"))
     (pad "2" thru_hole oval locked (at 2.5 0 270) (size 1.7 2) (drill 1) (layers *.Cu *.Mask)
@@
     (effects (font (size 3 3) (thickness 0.7)))
   )
+  (gr_text "power\noutput" (at 69.02 110.05) (layer "F.SilkS")
+    (effects (font (size 1 1) (thickness 0.25)))
+  )
+  (gr_text "made by:" (at 83.17 148.39) (layer "F.SilkS")
+    (effects (font (size 1 1) (thickness 0.25)))
+  )
   (gr_text "Olivia & Andrew 2022" (at 100.21 148.13) (layer "F.SilkS")
