File: cad-source-files/accessory-boards/servo_board/servo_board.kicad_pcb (KiCad board)
At the start: 2 copper layers, 50 x 22 mm, 18 parts, among them J1 Conn_01x02, J2 Conn_01x02, J4 Servo Header x2, J6 Conn_01x02, J9 Conn_01x06_MountingPin, Q1 LOW PWR FET, Q2 LOW PWR FET

Commit message: 12-2 boards ordered
Parts:
- J6: footprint Connector_JST:JST_XH_2_VERTICAL -> Connector_JST:JST_PH_B2B-PH-SM4-TB_1x02-1MP_P2.00mm_Vertical
- moved J6 4.57 mm to (170.3, 76.2), turned to -90 degrees
Routing:
- net GND: vias 87 -> 74
Other:
- board text added: "POWER INPUT"
