File: cad-source-files/accessory-boards/servo_board/servo_board.kicad_sch (KiCad schematic)
At the start: 18 parts, among them J1 Conn_01x02, J2 Conn_01x02, J4 Servo Header x2, J6 Conn_01x02, J9 Conn_01x06_MountingPin, Q1 LOW PWR FET, Q2 LOW PWR FET

Commit message: 12-2 boards ordered
Parts:
- J6: footprint Connector_JST:JST_XH_2_VERTICAL -> Connector_JST:JST_PH_B2B-PH-SM4-TB_1x02-1MP_P2.00mm_Vertical
Other:
- moved on the sheet: C1, D1, D2, D3, D4, J1, J2, J4, J6, Q1, Q2, R1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
