File: cad-source-files/joypad/joypad.kicad_sch (KiCad schematic)
At the start: 78 parts, among them J2 ftdi_conn, J4 Conn_01x04, J5 Conn_01x04, SW1 SW_Push, SW10 SW_Push, SW11 SW_Push, SW12 SW_Push, SW2 SW_Push, SW3 SW_Push, SW4 SW_Push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

Commit message: jerry!
Parts:
- removed C1: .1uF 100V, Capacitor_SMD:C_0805_2012Metric, symbol Device:C_Small
- removed C14, C2, C5: .1uF, Capacitor_SMD:C_0603_1608Metric, symbol Device:C_Small
- removed C15: 22uF, Capacitor_SMD:C_0805_2012Metric, symbol Device:C_Small
- removed C3: 4.7uF 100V, Capacitor_SMD:C_0805_2012Metric, symbol Device:C_Small
- removed C4: .1uF 100V, Capacitor_SMD:C_0805_2012Metric, symbol Device:CP_Small
- removed C6: 22uF, Capacitor_SMD:C_0805_2012Metric, symbol Device:CP_Small
- removed D7: D_TVS_x2_AAC, Package_TO_SOT_SMD:SOT-23, symbol Device:D_TVS_x2_AAC
- removed H10, H11, H6, H7, H8, H9: MountingHole, MountingHole:MountingHole_2.5mm_Pad, symbol Mechanical:MountingHole
- removed J4, J5: Conn_01x04, Connector_JST:JST_PH_S4B-PH-SM4-TB_1x04-1MP_P2.00mm_Horizontal, symbol Connector_Generic_MountingPin:Conn_01x04_MountingPin
- removed L1: 22uH, EvezorLIB:INDUCTOR_7.5X6.6_GCDA0630-220MC, symbol Device:L
- removed R1: 10k, Resistor_SMD:R_0603_1608Metric, symbol Device:R_Small
- removed R2: 82k, Resistor_SMD:R_0603_1608Metric, symbol Device:R_Small
- removed TP1, TP10, TP2, TP3, TP4, TP5, TP6, TP7, TP8, TP9: TestPoint, Evezor_extras:TestPoint_THTPad_D1.0mm_Drill0.5mm, symbol Connector:TestPoint
- removed U1: SY8401ABC, Package_TO_SOT_SMD:SOT-23-6, symbol Evezor_Library:REGULATOR_VOLTAGE_HT7463A
- removed U5: Trans_CAN_SN65HVD230DR, EvezorLIB:CAN-TRANS-SN65HVD230DR, symbol Evezor_Library:Trans_CAN_SN65HVD230DR
- added J1: Conn_01x04, Connector_PinSocket_2.54mm:PinSocket_1x04_P2.54mm_Vertical, symbol Connector_Generic:Conn_01x04
- added J3: Barrel_Jack, Connector_BarrelJack:BarrelJack_Horizontal, symbol Connector:Barrel_Jack
- J2: footprint Evezor_extras:CONN-SH-6P-VERTICAL -> Connector_JST:JST_SH_SM06B-SRSS-TB_1x06-1MP_P1.00mm_Horizontal
- SW1, SW11, SW12, SW2, SW3, SW4, SW5, SW6: footprint EvezorLIB:SWITCH_2x3_SMD_TACTILE_GREEN -> Button_Switch_SMD:SWITCH_2x3_SMD_TACTILE_GREEN
- U3: footprint Evezor_extras:ESP32-WROOM-32U -> RF_Module:ESP32-WROOM-32U_evezor
Connections:
- net VREG_OUT is gone; now on an unnamed net: U2.3 (VI)
- net +3V3: now also D8.2 (A), J1.1 (Pin_1)
- net BLUE: no longer U3.12 (A2-IO27)
- net DOWN: no longer U3.37 (VMOSI-IO23)
- net GND: now also J1.2 (Pin_2), J3.2; no longer D1.2 (A)
- net GREEN: no longer U3.10 (SCL1-DAC1-A2-IO25)
- net HBT_LED: no longer U3.29 (IO5)
- net JOY_SW_1: no longer U3.30 (SCL0-VCLK-IO18)
- net JOY_SW_2: no longer U3.13 (HSCK-A2-IO14)
- net LEFT: no longer U3.31 (SDA0-VMISO-IO19)
- net NEO_BAR: no longer U3.14 (HMISO-A2-IO12)
- net NEO_STATUS: no longer U3.28 (IO17)
- net RED: no longer U3.11 (SDA1-DAC2-A2-IO26)
- net RIGHT: no longer U3.36 (IO22)
- net SELECT: no longer U3.23 (A2-IO15)
- net START: no longer U3.16 (HMOSI-A2-IO13)
- net UP: no longer U3.33 (IO21)
- net VBUS: now also D1.2 (A), J3.1; no longer D2.2 (A), J2.5 (Pin_5)
- net YELLOW: no longer U3.9 (A1-IO33)
- net at D1.1 (K): now also D2.1 (K)
- net CAN_RX: no longer names the net of U3.27 (IO16)
- net CAN_SLP: no longer names the net of U3.24 (A2-IO2)
- net CAN_TX: no longer names the net of U3.26 (A2-IO4)
- removed net PWR: D2.1 (K), D8.2 (A)
- new net +5V: D2.2 (A), J2.5 (Pin_5)
- new net LCD_SCL: J1.3 (Pin_3)
- new net LCD_SDA: J1.4 (Pin_4)
- no-connect marks 9 -> 8
Other:
- note added: "LCD"
- note added: "STACHE STATION RESET"
- note removed: "CAN"
- note removed: "STATUS LEDS FUNCTION BUTTON BOOT/ RESET"
- moved on the sheet: D2

Commit message: things are connected but theres still more things to be done
Connections:
- net BLUE: now also U3.30 (SCL0-VCLK-IO18)
- net DOWN: now also U3.11 (SDA1-DAC2-A2-IO26)
- net GREEN: now also U3.29 (IO5)
- net HBT_LED: now also U3.24 (A2-IO2)
- net JOY_SW_1: now also U3.9 (A1-IO33)
- net JOY_SW_2: now also U3.28 (IO17)
- net LCD_SCL: now also U3.37 (VMOSI-IO23)
- net LCD_SDA: now also U3.36 (IO22)
- net LEFT: now also U3.10 (SCL1-DAC1-A2-IO25)
- net NEO_BAR: now also U3.23 (A2-IO15)
- net NEO_STATUS: now also U3.16 (HMOSI-A2-IO13)
- net RED: now also U3.33 (IO21)
- net RIGHT: now also U3.13 (HSCK-A2-IO14)
- net SELECT: now also U3.14 (HMISO-A2-IO12)
- net START: now also U3.27 (IO16)
- net UP: now also U3.12 (A2-IO27)
- net YELLOW: now also U3.31 (SDA0-VMISO-IO19)
Changed lines of the file:
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@@
     (effects (font (size 2.0066 2.0066)) (justify left bottom))
   )
-  (label "LCD_SCL" (at 340.36 162.56 180)
+  (label "LCD_SCL" (at 316.23 182.88 180)
     (effects (font (size 1.27 1.27)) (justify right bottom))
   )
@@
     (effects (font (size 1.27 1.27)) (justify right bottom))
   )
-  (label "JOY_SW_2" (at 340.36 157.48 180)
+  (label "JOY_SW_2" (at 316.23 170.18 180)
     (effects (font (size 1.27 1.27)) (justify right bottom))
   )
@@
     (effects (font (size 1.27 1.27)) (justify left bottom))
   )
-  (label "SELECT" (at 340.36 160.02 180)
+  (label "SELECT" (at 313.69 157.48 180)
     (effects (font (size 1.27 1.27)) (justify right bottom))
   )
-  (label "START" (at 340.36 154.94 180)
+  (label "START" (at 311.15 167.64 180)
     (effects (font (size 1.27 1.27)) (justify right bottom))
   )
@@
     (effects (font (size 1.27 1.27)) (justify left bottom))
   )
-  (label "RIGHT" (at 342.9 175.26 180)
+  (label "RIGHT" (at 313.69 162.56 180)
     (effects (font (size 1.27 1.27)) (justify right bottom))
   )
@@
     (effects (font (size 1.27 1.27)) (justify left bottom))
   )
-  (label "DOWN" (at 342.9 177.8 180)
+  (label "DOWN" (at 316.23 187.96 180)
     (effects (font (size 1.27 1.27)) (justify right bottom))
   )
@@
     (effects (font (size 1.27 1.27)) (justify left bottom))
   )
-  (label "HBT_LED" (at 339.09 149.86 180)
+  (label "HBT_LED" (at 312.42 147.32 180)
     (effects (font (size 1.27 1.27)) (justify right bottom))
   )
@@
     (effects (font (size 1.27 1.27)) (justify left bottom))
   )
-  (label "UP" (at 342.9 172.72 180)
+  (label "UP" (at 316.23 190.5 180)
     (effects (font (size 1.27 1.27)) (justify right bottom))
   )
@@
     (effects (font (size 1.27 1.27)) (justify right bottom))
   )
-  (label "LCD_SDA" (at 339.09 147.32 180)
+  (label "LCD_SDA" (at 316.23 180.34 180)
     (effects (font (size 1.27 1.27)) (justify right bottom))
   )
@@
     (effects (font (size 1.27 1.27)) (justify left bottom))
   )
-  (label "LEFT" (at 342.9 170.18 180)
+  (label "LEFT" (at 316.23 185.42 180)
     (effects (font (size 1.27 1.27)) (justify right bottom))
   )
-  (label "YELLOW" (at 341.63 187.96 180)
+  (label "YELLOW" (at 316.23 175.26 180)
     (effects (font (size 1.27 1.27)) (justify right bottom))
   )
-  (label "BLUE" (at 342.9 185.42 180)
+  (label "BLUE" (at 316.23 172.72 180)
     (effects (font (size 1.27 1.27)) (justify right bottom))
   )
@@
     (effects (font (size 1.27 1.27)) (justify left bottom))
   )
-  (label "NEO_BAR" (at 340.36 152.4 180)
+  (label "NEO_BAR" (at 313.69 165.1 180)
     (effects (font (size 1.27 1.27)) (justify right bottom))
   )
@@
     (effects (font (size 1.27 1.27)) (justify left bottom))
   )
-  (label "JOY_SW_1" (at 342.9 167.64 180)
+  (label "JOY_SW_1" (at 316.23 195.58 180)
     (effects (font (size 1.27 1.27)) (justify right bottom))
   )
-  (label "GREEN" (at 342.9 180.34 180)
+  (label "GREEN" (at 312.42 154.94 180)
     (effects (font (size 1.27 1.27)) (justify right bottom))
   )
@@
     (effects (font (size 1.27 1.27)) (justify left bottom))
   )
-  (label "RED" (at 342.9 182.88 180)
+  (label "RED" (at 316.23 177.8 180)
     (effects (font (size 1.27 1.27)) (justify right bottom))
   )
@@
     (effects (font (size 1.27 1.27)) (justify left bottom))
   )
-  (label "NEO_STATUS" (at 342.9 165.1 180)
+  (label "NEO_STATUS" (at 313.69 160.02 180)
     (effects (font (size 1.27 1.27)) (justify right bottom))
   )

Commit message: 12-2 boards ordered
Parts:
- SW10, SW7, SW8, SW9: footprint Evezor_BUTTONS:12mm_pushbutton -> Button_Switch_SMD:12mm_pushbutton
- U4, U6: footprint Evezor_BUTTONS:JOYSTICK -> Potentiometer_THT:JOYSTICK
Changed lines of the file:
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@@
     (property "Reference" "SW7" (id 0) (at 170.18 47.371 0))
     (property "Value" "SW_Push" (id 1) (at 170.18 49.6824 0))
-    (property "Footprint" "Evezor_BUTTONS:12mm_pushbutton" (id 2) (at 170.18 49.53 0)
+    (property "Footprint" "Button_Switch_SMD:12mm_pushbutton" (id 2) (at 170.18 49.53 0)
       (effects (font (size 1.27 1.27)) hide)
     )
@@
     (property "Reference" "SW10" (id 0) (at 170.18 105.791 0))
     (property "Value" "SW_Push" (id 1) (at 170.18 108.1024 0))
-    (property "Footprint" "Evezor_BUTTONS:12mm_pushbutton" (id 2) (at 170.18 107.95 0)
+    (property "Footprint" "Button_Switch_SMD:12mm_pushbutton" (id 2) (at 170.18 107.95 0)
       (effects (font (size 1.27 1.27)) hide)
     )
@@
     (property "Reference" "SW8" (id 0) (at 170.18 67.691 0))
     (property "Value" "SW_Push" (id 1) (at 170.18 70.0024 0))
-    (property "Footprint" "Evezor_BUTTONS:12mm_pushbutton" (id 2) (at 170.18 69.85 0)
+    (property "Footprint" "Button_Switch_SMD:12mm_pushbutton" (id 2) (at 170.18 69.85 0)
       (effects (font (size 1.27 1.27)) hide)
     )
@@
     (property "Reference" "U4" (id 0) (at 52.705 36.449 0))
     (property "Value" "JOYSTICK" (id 1) (at 52.705 38.7604 0))
-    (property "Footprint" "Evezor_BUTTONS:JOYSTICK" (id 2) (at 53.34 54.61 0)
+    (property "Footprint" "Potentiometer_THT:JOYSTICK" (id 2) (at 53.34 54.61 0)
       (effects (font (size 1.27 1.27)) hide)
     )
@@
     (property "Reference" "SW9" (id 0) (at 170.18 85.471 0))
     (property "Value" "SW_Push" (id 1) (at 170.18 87.7824 0))
-    (property "Footprint" "Evezor_BUTTONS:12mm_pushbutton" (id 2) (at 170.18 87.63 0)
+    (property "Footprint" "Button_Switch_SMD:12mm_pushbutton" (id 2) (at 170.18 87.63 0)
       (effects (font (size 1.27 1.27)) hide)
     )
@@
     (property "Reference" "U6" (id 0) (at 52.705 59.309 0))
     (property "Value" "JOYSTICK" (id 1) (at 52.705 61.6204 0))
-    (property "Footprint" "Evezor_BUTTONS:JOYSTICK" (id 2) (at 53.34 77.47 0)
+    (property "Footprint" "Potentiometer_THT:JOYSTICK" (id 2) (at 53.34 77.47 0)
       (effects (font (size 1.27 1.27)) hide)
     )
@@
     )
     (path "/03fbb8b0-7d92-45b2-90c4-df2e3cacbc1a"
-      (reference "SW7") (unit 1) (value "SW_Push") (footprint "Evezor_BUTTONS:12mm_pushbutton")
+      (reference "SW7") (unit 1) (value "SW_Push") (footprint "Button_Switch_SMD:12mm_pushbutton")
     )
     (path "/5a5cb507-5f5f-43e2-b1b0-c3c3cac1681a"
-      (reference "SW8") (unit 1) (value "SW_Push") (footprint "Evezor_BUTTONS:12mm_pushbutton")
+      (reference "SW8") (unit 1) (value "SW_Push") (footprint "Button_Switch_SMD:12mm_pushbutton")
     )
     (path "/e177a81e-4ab2-4bae-a8ae-c41575531892"
-      (reference "SW9") (unit 1) (value "SW_Push") (footprint "Evezor_BUTTONS:12mm_pushbutton")
+      (reference "SW9") (unit 1) (value "SW_Push") (footprint "Button_Switch_SMD:12mm_pushbutton")
     )
     (path "/47b78f3f-a4b5-4383-a1f4-6aa5230c8711"
-      (reference "SW10") (unit 1) (value "SW_Push") (footprint "Evezor_BUTTONS:12mm_pushbutton")
+      (reference "SW10") (unit 1) (value "SW_Push") (footprint "Button_Switch_SMD:12mm_pushbutton")
     )
     (path "/d1f283c1-9939-4441-9cff-12e7faf5d20b"
@@
     )
     (path "/693fc83f-c890-49a9-8969-38f2da9ec659"
-      (reference "U4") (unit 1) (value "JOYSTICK") (footprint "Evezor_BUTTONS:JOYSTICK")
+      (reference "U4") (unit 1) (value "JOYSTICK") (footprint "Potentiometer_THT:JOYSTICK")
     )
     (path "/f0f3818b-a4f9-4082-9223-bfd32fbc27ae"
-      (reference "U6") (unit 1) (value "JOYSTICK") (footprint "Evezor_BUTTONS:JOYSTICK")
-    )
-  )
+      (reference "U6") (unit 1) (value "JOYSTICK") (footprint "Potentiometer_THT:JOYSTICK")
+    )
+  )
